Commit message: project2 before summitting

File: PROJECT2/catkin_ws/src/my_robot/urdf/my_robot.xacro (robot description, xacro)
@@ -2,4 +2,5 @@
 <robot name="my_robot" xmlns:xacro="http://www.ros.org/wiki/xacro">
   <link name="robot_footprint"></link>
+  <xacro:include filename="$(find my_robot)/urdf/my_robot.gazebo" />
   <joint name="robot_footprint_joint" type="fixed">
     <origin xyz="0 0 0" rpy="0 0 0" />
@@ -30,5 +31,5 @@
       </geometry>
     </visual>
-    <collision name='collision'>
+    <collision name='back_caster_collision'>
       <origin xyz="-0.2 0 -0.1" rpy=" 0 0 0"/>
       <geometry>
@@ -42,5 +43,5 @@
       </geometry>
     </visual>
-    <collision name='collision'>
+    <collision name='front_caster_collision'>
       <origin xyz="0.2 0 -0.1" rpy=" 0 0 0"/>
       <geometry>
@@ -67,5 +68,5 @@
     </inertial>
     <collision name='collision'>
-      <origin xyz="0 0 0" rpy=" 0 0 0"/>
+      <origin xyz="0 0 0" rpy=" 0 1.5707 1.5707"/>
       <geometry>
         <cylinder radius="0.1" length="0.06"/>
@@ -73,5 +74,5 @@
     </collision>
     <visual name='left_wheel_visual'>
-      <origin xyz="0 0 0" rpy=" 0 0 0"/>
+      <origin xyz="0 0 0" rpy=" 0 1.5707 1.5707"/>
       <geometry>
         <cylinder radius="0.1" length="0.06"/>
@@ -91,5 +92,5 @@
     </inertial>
     <collision name='right_wheel_collision'>
-      <origin xyz="0 0 0" rpy=" 0 0 0"/>
+      <origin xyz="0 0 0" rpy=" 0 1.5707 1.5707"/>
       <geometry>
         <cylinder radius="0.1" length="0.06"/>
@@ -97,5 +98,5 @@
     </collision>
     <visual name='right_wheel_visual'>
-      <origin xyz="0 0 0" rpy=" 0 0 0"/>
+      <origin xyz="0 0 0" rpy="0 1.5707 1.5707"/>
       <geometry>
         <cylinder radius="0.1" length="0.06"/>
@@ -104,5 +105,5 @@
   </link>
   <joint type="continuous" name="left_wheel_hinge">
-    <origin xyz="0.2 -.26 -0.15" rpy="0 0 0"/>
+    <origin xyz="0.2 -.23 -0.1" rpy="0 0 0"/>
     <child link="left_wheel"/>
     <parent link="chassis"/>
@@ -112,5 +113,5 @@
   </joint>
   <joint type="continuous" name="right_wheel_hinge">
-    <origin xyz="0.2 .26 -0.15" rpy="0 0 0"/>
+    <origin xyz="0.2 .23 -0.1" rpy="0 0 0"/>
     <child link="right_wheel"/>
     <parent link="chassis"/>
@@ -183,3 +184,15 @@
     <dynamics damping="1.0" friction="1.0"/>
   </joint>
+  <gazebo reference="right_wheel_hinge">
+      <material>Gazebo/Blue</material>
+  </gazebo>
+  <gazebo reference="left_wheel_hinge">
+      <material>Gazebo/Blue</material>
+  </gazebo>
+  <gazebo reference="chassis">
+      <material>Gazebo/Yellow</material>
+  </gazebo>
+  <gazebo reference="hokuyo">
+      <material>Gazebo/Red</material>
+  </gazebo>
 </robot>

Commit message: Robot dimensions modification

File: PROJECT2/catkin_ws/src/my_robot/urdf/my_robot.xacro (robot description, xacro)
@@ -105,5 +105,5 @@
   </link>
   <joint type="continuous" name="left_wheel_hinge">
-    <origin xyz="0.2 -.23 -0.1" rpy="0 0 0"/>
+    <origin xyz="-0.2 -.23 -0.1" rpy="0 0 0"/>
     <child link="left_wheel"/>
     <parent link="chassis"/>
@@ -113,5 +113,5 @@
   </joint>
   <joint type="continuous" name="right_wheel_hinge">
-    <origin xyz="0.2 .23 -0.1" rpy="0 0 0"/>
+    <origin xyz="-0.2 .23 -0.1" rpy="0 0 0"/>
     <child link="right_wheel"/>
     <parent link="chassis"/>
